Commit message: Changed realsense to pc4, added etc env variable, add joint temp ui

File: src/tmms_description/urdf/tmms_description.urdf.xacro (robot description, xacro)
@@ -1,4 +1,4 @@
 <?xml version='1.0' encoding='utf-8'?>
-<robot name="tmms_description">
+<robot name="tmms_description" xmlns:xacro="http://www.ros.org/wiki/xacro">
   <link name="base_link">
     <inertial>
@@ -65,5 +65,5 @@
     <axis xyz="0 0 0" />
   </joint>
-  <link name="imu_link">
+  <link name="dog_imu_link">
     <inertial>
       <origin xyz="-2.02E-17 1.73E-17 -1.39E-17" rpy="0 0 0" />
@@ -75,5 +75,5 @@
     <origin xyz="0 -0.02341 0.04927" rpy="0 0 0" />
     <parent link="base_link" />
-    <child link="imu_link" />
+    <child link="dog_imu_link" />
     <axis xyz="0 0 0" />
   </joint>
@@ -814,3 +814,11 @@
     <axis xyz="0 0 0" />
   </joint>
+  <link name="camera_front_link" />
+  <joint name="joint_camera_front" type="fixed">
+    <origin xyz="$(env FRONT_REALSENSE_X) $(env FRONT_REALSENSE_Y) $(env FRONT_REALSENSE_Z)"
+            rpy="$(env FRONT_REALSENSE_ROLL) $(env FRONT_REALSENSE_PITCH) $(env FRONT_REALSENSE_YAW)" />
+    <parent link="rslidar" />
+    <child link="camera_front_link" />
+    <axis xyz="0 0 0" />
+  </joint>
 </robot>
